Commit message: Imported upstream version '0.2.1' of 'upstream'

File: magni_description/urdf/basic_magni.urdf (robot description, URDF)
Before this commit: robot magni, 4 links, 3 joints
Joints:
- joint raspicam_joint: origin xyz=0.035 0.145 0.14 rpy=0 0 3.1416 -> xyz=0.035 0.145 0.14 rpy=1.15191731 0 1.5707
